File: main.brd (EAGLE design)
At the start: 160 x 100 mm, 181 parts, among them J301 12401948E412A, Q101 IPP65R095C7, Q201 IPP65R190C7, Q202 IPP65R190C7, Q203 SiR182DP, Q204 SiR182DP, Q301 ISZ0702NLS, Q302 ISZ0702NLS, Q303 ISZ0702NLS, Q304 ISZ0702NLS, T201 706µH 41:4:4:4, U101 UCC28056B, U201 UCC256404, U202 TLV431E5, U203 UCC24624, U301 MAX25432

Commit message: Added firmware base, layout in progress
Parts:
- added C401: 33µF, rcl:C1206
- added C402, C403, C418: 10µF, rcl:C0805
- added C404, C407, C408, C410, C413, C414, C415, C431: 100nF, rcl:C0603
- added C405, C411, C412: 1µF, rcl:C0603
- added C406: 10nF, rcl:C0603
- added C409: 4.7µF, rcl:C0603
- added C416: 33nF, rcl:C0603
- added C417: 470nF, rcl:C0603
- added C419, C421, C423, C426: 82µF, rcl:E3,5-8
- added C420, C422: 270pF, rcl:C0603
- added C424: 0pF, rcl:C0603
- added C425: 18pF, rcl:C0603
- added C427: ?pF, rcl:C0603
- added C428: 0nF, rcl:C0603
- added C429: 1.2nF, rcl:C0603
- added C430: ?nF, rcl:C0603
- added C501, C504: 10µF 35V, rcl:C1206
- added C502, C503, C505, C506, C507, C508, C509, C510, C511, C512: 0.1µF, rcl:C0603
- added C513, C514: 22µF, rcl:C0805
- added C515, C516: 7pF, rcl:C0603
- added C517: 2.2µF, rcl:C0805
- added C518: 330µF, rcl:PANASONIC_D
- added D401, D402: NSR0530H, BW-Active:SOD323
- added J401: 12401948E412A, BW-Connectors:12401948E412A
- added J501: ICSP, BW-Connectors:5PIN-1.27
- added J502: UART, pinhead:1X02
- added L401: 4.7µH, BW-PassiveMechanical:B82559B*A016
- added L501: 10µH, BW-PassiveMechanical:RLB0912
- added LSP101: AC_L, solpad:LSP13
- added LSP102: AC_N, solpad:LSP13
- added Q401, Q402, Q403, Q404: ISZ0702NLS, BW-Active:TSDSON-8
- added R236: 7.5kΩ, rcl:R0603
- added R237, R317, R403, R408, R409, R410, R412, R417: 0Ω, rcl:R0603
- added R316, R416: 62kΩ, rcl:R0603
- added R318, R401, R418: 5mΩ, rcl:R0805
- added R319, R419: 100kΩ?, rcl:R0603
- added R402, R404: 4.7kΩ, rcl:R0603
- added R405: 2.2kΩ, rcl:R0603
- added R406: 100kΩ, rcl:R0603
- added R407: 1kΩ, rcl:R0603
- added R411: 1MΩ, rcl:R0603
- added R413: 3mΩ, rcl:R0805
- added R414: 499Ω, rcl:R0603
- added R415: ?Ω, rcl:R0603
- added R501: 10kΩ, resistor:R0603
- added R502: 1kΩ, resistor:R0603
- added R503, R505: 100kΩ, resistor:R0603
- added R504: 8.2kΩ, resistor:R0603
- added R506: 20kΩ, resistor:R0603
- added R507: 0Ω, resistor:R0603
- added SJ501, SJ502, SJ503, SJ504: (no value), jumper:SJ
- added U401: MAX25432, BW-Active:TQFN-40
- added U501: TPS54308, BW-Active:SOT23-6L
- added U502: PIC32MZ-EF-064, BW-Active:TQFP64-10X10X1MM
- added U503: LD39150DT33, BW-Active:DFN6
- added XDS501: NHD-3.5-320240FT-FPCV, BW-Active:FFC3A20-20
- added Y501: 24MHz, BW-PassiveMechanical:XRCGB
- C211: value 10µF -> 22µF
- C213: value 330nF -> 3.3µF; device rcl:C0603 -> rcl:C0805
- R229: value ?Ω -> 0Ω
- R230: value 100Ω -> ?Ω
- R231: value 1kΩ -> 100Ω
- R232: value 470kΩ -> 0Ω
- R233: value 100kΩ -> 1kΩ
- R234: value 7.5kΩ -> 470kΩ
- R235: value 0Ω -> 100kΩ
- R303: value 4.7kΩ -> 0Ω
- R304: value 2.2kΩ -> 4.7kΩ
- R305: value 100kΩ -> 2.2kΩ
- R306: value 1kΩ -> 100kΩ
- R307: value 0Ω -> 1kΩ
- R308: value 1MΩ -> 0Ω
- R309: value 3mΩ -> 0Ω; device rcl:R0805 -> rcl:R0603
- R310: value 499Ω -> 0Ω
- R311: value ?Ω -> 1MΩ
- R312: value 62kΩ -> 0Ω
- R313: value 0Ω -> 3mΩ; device rcl:R0603 -> rcl:R0805
- R314: value 5mΩ -> 499Ω; device rcl:R0805 -> rcl:R0603
- R315: value 100kΩ? -> ?Ω
- moved Q304 277.1 mm to (79.0, 18.0), turned to 180 degrees
- moved Q303 275.9 mm to (74.0, 22.2)
- moved C315 273.3 mm to (75.9, 14.5), turned to 270 degrees
- moved C318 268.7 mm to (81.1, 15.0), flipped to the bottom, turned to 180 degrees
- moved C321 261.3 mm to (88.7, 4.50), turned to 270 degrees
- moved U301 260.8 mm to (66.7, 29.0), turned to 270 degrees
- moved C331 258.2 mm to (81.5, 8.30), flipped to the bottom, turned to 180 degrees
- moved C326 257.4 mm to (71.0, 11.5), turned to 180 degrees
- moved C301 257.2 mm to (82.0, 43.3), flipped to the bottom, turned to 180 degrees
- moved J301 255.3 mm to (78.0, 0.00)
- moved L301 253.2 mm to (86.0, 29.0), turned to 270 degrees
- moved C303 252.6 mm to (81.4, 43.3)
- moved R309 252.1 mm to (69.7, 34.5)
- moved C113 251.4 mm to (39.8, 36.5), flipped to the bottom
- moved C323 251.4 mm to (66.4, 4.40), turned to 180 degrees
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Connections:
- new net 3.3V_BULKR: C518.+, R507.1
- new net 3.6V: C513.1, C514.1, L501.2, R505.2, U503.2, U503.3
- new net LCD_!CS: U502.21, XDS501.A6, XDS501.B6
- new net LCD_!INT: U502.18, XDS501.A7, XDS501.B7
- new net LCD_!PD: U502.17, XDS501.A8, XDS501.B8
- new net LCD_MISO: U502.23, XDS501.A4, XDS501.B4
- new net LCD_MOSI: U502.22, XDS501.A5, XDS501.B5
- new net LCD_SCK: U502.29, XDS501.A3, XDS501.B3
- new net LLC_SR_VG1_R: Q203.4, R228.1
- new net LLC_SR_VG2_R: Q204.4, R232.2
- new net N$1: J502.2, U502.5
- new net N$2: J502.1, U502.6
- new net PIC_!MCLR: J501.1, R502.1, U502.9
- new net PIC_!MCLR!_FILTER: C502.1, R501.1, R502.2
- new net PIC_D+: SJ501.1, SJ503.1, U502.37
- new net PIC_D-: SJ502.1, SJ504.1, U502.36
- new net PIC_OSC1: C515.1, U502.31, Y501.1
- new net PIC_OSC2: C516.1, U502.32, Y501.3
- new net PIC_PGEC: J501.5, U502.15
- new net PIC_PGED: J501.4, U502.16
- new net PIC_VIN_SENSE: C503.1, R503.1, R504.2, U502.11
- new net PRELIN_BOOT: C509.1, U501.6
- new net PRELIN_FB: R505.1, R506.2, U501.4
- new net PRELIN_SW: C509.2, L501.1, U501.2
- new net PRI_DUMMY_1: T201.2
- new net PRI_DUMMY_2: T201.6
- new net USB1_DH1_R: Q301.4, R303.2, R305.1
- new net USB1_DH2_R: Q304.4, R312.2
- new net USB1_DL1_R: Q302.4, R309.2
- new net USB1_DL2_R: Q303.4, R310.2
- new net USB2_!ALERT: R406.2, U401.20, U502.49
- new net USB2_ADDR: R408.2, U401.34
- new net USB2_BIAS: C409.1, C410.1, D401.2, D402.2, U401.29
- new net USB2_BST1: C413.2, D401.1, U401.1
- new net USB2_BST2: C414.1, D402.1, U401.36
- new net USB2_CC1: C420.1, J401.A5, U401.25
- new net USB2_CC2: C422.1, J401.B5, U401.24
- new net USB2_CSN1: Q401.5-8, R401.2, U401.4
- new net USB2_CSP2: C415.1, Q404.5-8, R413.1, U401.33
- new net USB2_DH1: R403.1, U401.40
- new net USB2_DH1_R: Q401.4, R403.2, R405.1
- new net USB2_DH2: R412.1, U401.37
- new net USB2_DH2_R: Q404.4, R412.2
- new net USB2_DL1: R409.1, U401.2
- new net USB2_DL1_R: Q402.4, R409.2
- new net USB2_DL2: R410.1, U401.35
- new net USB2_DL2_R: Q403.4, R410.2
- new net USB2_DM: SJ504.2, U401.19
- new net USB2_DP: SJ503.2, U401.18
- new net USB2_EN: R407.1, U502.52
- new net USB2_GDRV: R411.1, U401.8
- new net USB2_HVDM: J401.A7, J401.B7, U401.21
- new net USB2_HVDP: J401.A6, J401.B6, U401.22
- new net USB2_HVEN: R407.2, U401.6
- new net USB2_ICOMP: C416.2, R414.1, U401.30
- new net USB2_ICOMP_R: C417.2, R414.2
- new net USB2_LX1: C413.1, L401.1, Q401.1, Q401.2, Q401.3, Q402.5-8, R405.2, U401.39
- new net USB2_LX2: C414.2, L401.2, Q403.5-8, Q404.1, Q404.2, Q404.3, U401.38
- new net USB2_OUT: C418.1, C419.+, C421.+, C423.+, C426.+, R413.2, R418.1, U401.32
- new net USB2_SCL: R402.2, U401.11, U502.51
- new net USB2_SDA: R404.2, U401.12, U502.50
- new net USB2_VBUS: C431.1, J401.A4B9, J401.B4A9, R418.2, R419.2, U401.31
- new net USB2_VCOMP: C424.1, C425.1, R415.1, R416.1, U401.27
- new net USB2_VCOMP_CPI: C424.2, C425.2, C427.1
- new net USB2_VCOMP_CZI: C428.2, C429.2, C430.1
- new net USB2_VCOMP_R: C428.1, C429.1, R417.2
- new net USB2_VCOMP_RI: R415.2, R416.2, R417.1
- new net USB2_VDD_BMC: C412.1, U401.13
- new net USB2_VDD_USB: C411.1, U401.17
- net 18V: now also C401.1, C403.1, C405.1, C407.1, C408.1, C501.1, C504.1, R401.1, R503.2, U401.28, U401.5, U501.3
- net 3.3V: now also C402.1, C404.1, C406.1, C505.1, C506.1, C507.1, C508.1, C510.1, C511.1, C512.1, C517.1, J501.2, R304.1, R306.1, R402.1, R404.1, R406.1, R501.2, R507.2, U401.16, U401.9, U502.19, U502.26, U502.34, U502.39, U502.54, U502.60, U502.8, U503.4, U503.5, XDS501.A1, XDS501.A17, XDS501.A18, XDS501.B1, XDS501.B17, XDS501.B18; no longer R303.1, R305.1
- net AC_L: now also LSP101.MP
- net AC_N: now also LSP102.MP
- net LLC_FB_COMP: now also R231.2; no longer R229.2
- net LLC_FB_COMPR: now also R229.2, R231.1; no longer R228.2, R229.1
- net LLC_FB_OPAP: now also R233.1; no longer R231.1
- net LLC_FB_OPK: now also R229.1; no longer R228.1
- net LLC_FB_VREF: now also R235.1, R236.2; no longer R232.2, R233.1
- net LLC_FB_VREFR: now also R236.1, R237.2; no longer R232.1, R235.2
- net LLC_OUT: now also R235.2; no longer R231.2
- net LLC_SR_VG1: now also R228.2; no longer Q203.4
- net LLC_SR_VG2: now also R232.1; no longer Q204.4
- net SGND: now also C401.2, C402.2, C403.2, C404.2, C405.2, C406.2, C407.2, C408.2, C409.2, C410.2, C411.2, C412.2, C415.2, C416.1, C417.1, C418.2, C419.-, C420.2, C421.-, C422.2, C423.-, C426.-, C427.2, C430.2, C431.2, C501.2, C502.2, C503.2, C504.2, C505.2, C506.2, C507.2, C508.2, C510.2, C511.2, C512.2, C513.2, C514.2, C515.2, C516.2, C517.2, C518.-, J401.A1B12, J401.B1A12, J401.M1, J401.M2, J401.M3, J401.M4, J501.3, Q402.1, Q402.2, Q402.3, Q403.1, Q403.2, Q403.3, R237.1, R308.1, R311.2, R319.1, R408.1, R411.2, R419.1, R504.1, R506.1, U401.23, U401.26, U401.3, U401.7, U401.EP, U501.1, U502.20, U502.25, U502.35, U502.40, U502.55, U502.59, U502.7, U503.1, U503.T, XDS501.A19, XDS501.A2, XDS501.A20, XDS501.B19, XDS501.B2, XDS501.B20; no longer R235.1, R307.1, R308.2, R315.1
- net USB1_!ALERT: now also R306.2, U502.42; no longer R305.2
- net USB1_ADDR: now also R308.2; no longer R307.2
- net USB1_CSP2: now also R313.1; no longer R309.1
- net USB1_DH1: now also R303.1; no longer Q301.4, R304.1
- net USB1_DH2: now also R312.1; no longer Q304.4
- net USB1_DL1: now also R309.1; no longer Q302.4
- net USB1_DL2: now also R310.1; no longer Q303.4
- net USB1_DM: now also SJ502.2
- net USB1_DP: now also SJ501.2
- net USB1_EN: now also R307.1, U502.45; no longer R306.1
- net USB1_GDRV: now also R311.1; no longer R308.1
- net USB1_HVEN: now also R307.2; no longer R306.2
- net USB1_ICOMP: now also R314.1; no longer R310.1
- net USB1_ICOMP_R: now also R314.2; no longer R310.2
- net USB1_LX1: now also R305.2; no longer R304.2
- net USB1_OUT: now also R313.2, R318.1; no longer R309.2, R314.1
- net USB1_SCL: now also U502.44
- net USB1_SDA: now also R304.2, U502.43; no longer R303.2
- net USB1_VBUS: now also R318.2, R319.2; no longer R314.2, R315.2
- net USB1_VCOMP: now also R315.1, R316.1; no longer R311.1, R312.1
- net USB1_VCOMP_R: now also R317.2; no longer R313.2
- net USB1_VCOMP_RI: now also R315.2, R316.2, R317.1; no longer R311.2, R312.2, R313.1
- net USB_SYNC: now also U401.10
Routing:
- net PGND: track 0.00 -> 64.5 mm, vias 0 -> 39
- net LLC_RVCC: track 0.00 -> 61.7 mm, vias 0 -> 3
- net LLC_FB_OPK: track 0.00 -> 54.6 mm
- net USB1_OUT: track 0.00 -> 53.8 mm, vias 0 -> 2
- net 18V: track 0.00 -> 43.6 mm, vias 0 -> 4
- net USB1_VBUS: track 0.00 -> 39.4 mm, vias 0 -> 8
- net LLC_BLK: track 0.00 -> 39.0 mm, vias 0 -> 1
- net LLC_PRI_OUT: track 0.00 -> 37.6 mm
- net LLC_BW: track 0.00 -> 37.5 mm, vias 0 -> 1
- net LLC_ISNS: track 0.00 -> 36.6 mm, vias 0 -> 1
- net LLC_HV: track 0.00 -> 36.6 mm, vias 0 -> 1
- net LLC_VCC: track 0.00 -> 36.5 mm, vias 0 -> 2
- net USB1_HVDM: track 0.00 -> 35.5 mm
- net LLC_FB_OPA: track 0.00 -> 34.9 mm
- net USB1_HVDP: track 0.00 -> 34.5 mm
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- added copper zone on layer 1, net 370V
- added copper zone on layer 1, net AC_L_FILTERED
- added copper zone on layer 1, net AC_L_FUSED
- added copper zone on layer 1, net AC_N
- added copper zone on layer 1, net AC_N_FILTERED
- added copper zone on layer 1, net AC_RECTIFIED
- added copper zone on layer 16, net LLC_HS
- added copper zone on layer 16, net LLC_OUT
- added copper zone on layer 1, net LLC_SR_VD1
- added copper zone on layer 16, net LLC_SR_VD1
- added copper zone on layer 1, net LLC_SR_VD2
- added copper zone on layer 16, net LLC_SR_VD2
- added copper zone on layer 16, net PFC_SW_NODE
- added copper zone on layer 1, net PGND
- added copper zone on layer 16, net PGND
- added copper zone on layer 1, net SGND
- added copper zone on layer 16, net SGND
- added copper zone on layer 1, net USB1_CSN1
- added copper zone on layer 16, net USB1_CSN1
- added copper zone on layer 1, net USB1_CSP2
- added copper zone on layer 16, net USB1_CSP2
- added copper zone on layer 1, net USB1_LX1
- added copper zone on layer 1, net USB1_LX2
Other:
- outline, holes or cut-outs redrawn
- board text added: "<- FPC Center NHD"

Commit message: Supply PCB done (?)
Parts:
- added TP101, TP201, TP202, TP301, TP302, TP303, TP304, TP305, TP306, TP401, TP402, TP403, TP404, TP405, TP406, TP501, TP502, TP503, TP504, TP505, TP506, TP507, TP508, TP509: RCU-0(J), BW-PassiveMechanical:TP_0603_JOINED
- C502, C503, C505, C506, C507, C508, C509, C510, C511, C512: value 0.1µF -> 100nF
- moved C419 273.1 mm to (128.9, 12.1)
- moved C403 268.4 mm to (125.4, 43.3)
- moved L401 267.9 mm to (130.0, 29.0), turned to 270 degrees
- moved C421 267.3 mm to (132.7, 4.50), turned to 270 degrees
- moved R405 263.3 mm to (127.0, 40.0), turned to 270 degrees
- moved C418 263.2 mm to (125.1, 15.0), flipped to the bottom, turned to 180 degrees
- moved C413 260.9 mm to (117.9, 32.3), turned to 270 degrees
- moved Q402 260.2 mm to (118.0, 35.8)
- moved C503 254.3 mm to (147.2, 8.70), flipped to the bottom, turned to 270 degrees
- moved C414 254.0 mm to (117.9, 25.6), turned to 270 degrees
- moved J502 253.0 mm to (141.9, 7.30), turned to 180 degrees
- moved C416 252.4 mm to (109.4, 20.9), turned to 90 degrees
- moved C422 252.1 mm to (108.7, 13.8), turned to 180 degrees
- moved Q403 251.1 mm to (118.0, 22.2)
- moved C425 250.5 mm to (113.4, 16.1), flipped to the bottom, turned to 270 degrees
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Connections:
- net N$1 renamed PIC_UART_TX
- net N$2 renamed PIC_UART_RX
- net 18V: now also TP201.1
- net 3.3V: now also TP501.1
- net 3.6V: now also TP509.1
- net 370V: now also TP101.1
- net LCD_!CS: now also TP506.1
- net LCD_!INT: now also TP507.1
- net LCD_!PD: now also TP508.1
- net LCD_MISO: now also TP504.1
- net LCD_MOSI: now also TP505.1
- net LCD_SCK: now also TP503.1
- net PIC_VIN_SENSE: now also TP502.1
- net SGND: now also TP202.1
- net USB1_!ALERT: now also TP304.1
- net USB1_CC1: now also TP305.1
- net USB1_EN: now also TP301.1
- net USB1_SCL: now also TP302.1
- net USB1_SDA: now also TP303.1
- net USB1_VBUS: now also TP306.1
- net USB2_!ALERT: now also TP404.1
- net USB2_CC1: now also TP405.1
- net USB2_EN: now also TP401.1
- net USB2_SCL: now also TP402.1
- net USB2_SDA: now also TP403.1
- net USB2_VBUS: now also TP406.1
Routing:
- net 3.3V: track 17.1 -> 293.7 mm, vias 2 -> 18
- net USB1_!ALERT: track 1.60 -> 135.6 mm, vias 1 -> 2
- net USB1_DM: track 0.00 -> 129.3 mm
- net USB1_DP: track 0.00 -> 128.4 mm
- net USB1_SDA: track 8.11 -> 125.7 mm
- net USB1_SCL: track 4.00 -> 120.7 mm
- net USB1_EN: track 0.00 -> 106.7 mm
- net USB2_!ALERT: track 0.00 -> 86.5 mm, vias 0 -> 2
- net USB2_DM: track 0.00 -> 81.9 mm, vias 0 -> 2
- net USB2_DP: track 0.00 -> 80.7 mm, vias 0 -> 2
- net USB2_SDA: track 0.00 -> 77.3 mm
- net USB2_SCL: track 0.00 -> 73.0 mm
- net USB_SYNC: track 0.00 -> 62.2 mm, vias 0 -> 4
- net PIC_VIN_SENSE: track 0.00 -> 61.9 mm, vias 0 -> 4
- net USB2_EN: track 0.00 -> 60.0 mm
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- added copper zone on layer 1, net 18V
- added copper zone on layer 16, net 18V
- added copper zone on layer 1, net LOGO
- added copper zone on layer 1, net USB2_CSN1
- added copper zone on layer 16, net USB2_CSN1
- added copper zone on layer 1, net USB2_CSP2
- added copper zone on layer 16, net USB2_CSP2
- added copper zone on layer 1, net USB2_LX1
- added copper zone on layer 1, net USB2_LX2
Other:
- outline, holes or cut-outs redrawn
- board text added: "JLCJLCJLCJLC"
- board text added: "USB PD Supply ©2023 BlockWorker blockworker.de"
- board text added: "USB1"
- board text added: "USB2"

Commit message: Base design complete, adapter firmware started
Parts:
- D301, D302, D401, D402: value NSR0530H -> SS0840WS
Changed lines of the file:
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@@
 <grid distance="1" unitdist="mm" unit="mm" style="lines" multiple="1" display="no" altdistance="0.1" altunitdist="mm" altunit="mm"/>
 <layers>
-<layer number="1" name="Top" color="4" fill="1" visible="no" active="yes"/>
+<layer number="1" name="Top" color="4" fill="1" visible="yes" active="yes"/>
 <layer number="2" name="Route2" color="16" fill="1" visible="no" active="no"/>
 <layer number="3" name="Route3" color="17" fill="1" visible="no" active="no"/>
@@
 <layer number="19" name="Unrouted" color="6" fill="1" visible="yes" active="yes"/>
 <layer number="20" name="Dimension" color="24" fill="1" visible="yes" active="yes"/>
-<layer number="21" name="tPlace" color="7" fill="1" visible="no" active="yes"/>
+<layer number="21" name="tPlace" color="7" fill="1" visible="yes" active="yes"/>
 <layer number="22" name="bPlace" color="7" fill="1" visible="yes" active="yes"/>
-<layer number="23" name="tOrigins" color="15" fill="1" visible="no" active="yes"/>
+<layer number="23" name="tOrigins" color="15" fill="1" visible="yes" active="yes"/>
 <layer number="24" name="bOrigins" color="15" fill="1" visible="yes" active="yes"/>
-<layer number="25" name="tNames" color="7" fill="1" visible="no" active="yes"/>
+<layer number="25" name="tNames" color="7" fill="1" visible="yes" active="yes"/>
 <layer number="26" name="bNames" color="7" fill="1" visible="yes" active="yes"/>
-<layer number="27" name="tValues" color="7" fill="1" visible="no" active="yes"/>
+<layer number="27" name="tValues" color="7" fill="1" visible="yes" active="yes"/>
 <layer number="28" name="bValues" color="7" fill="1" visible="yes" active="yes"/>
-<layer number="29" name="tStop" color="7" fill="3" visible="no" active="yes"/>
+<layer number="29" name="tStop" color="7" fill="3" visible="yes" active="yes"/>
 <layer number="30" name="bStop" color="7" fill="6" visible="yes" active="yes"/>
 <layer number="31" name="tCream" color="7" fill="4" visible="no" active="yes"/>
@@
 <layer number="37" name="tTest" color="7" fill="1" visible="no" active="yes"/>
 <layer number="38" name="bTest" color="7" fill="1" visible="no" active="yes"/>
-<layer number="39" name="tKeepout" color="4" fill="11" visible="no" active="yes"/>
+<layer number="39" name="tKeepout" color="4" fill="11" visible="yes" active="yes"/>
 <layer number="40" name="bKeepout" color="1" fill="11" visible="yes" active="yes"/>
-<layer number="41" name="tRestrict" color="4" fill="10" visible="no" active="yes"/>
+<layer number="41" name="tRestrict" color="4" fill="10" visible="yes" active="yes"/>
 <layer number="42" name="bRestrict" color="1" fill="10" visible="yes" active="yes"/>
 <layer number="43" name="vRestrict" color="2" fill="10" visible="yes" active="yes"/>
 <layer number="44" name="Drills" color="7" fill="1" visible="no" active="yes"/>
 <layer number="45" name="Holes" color="7" fill="1" visible="yes" active="yes"/>
-<layer number="46" name="Milling" color="3" fill="1" visible="no" active="yes"/>
-<layer number="47" name="Measures" color="7" fill="1" visible="no" active="yes"/>
-<layer number="48" name="Document" color="7" fill="1" visible="no" active="yes"/>
-<layer number="49" name="Reference" color="7" fill="1" visible="no" active="yes"/>
+<layer number="46" name="Milling" color="3" fill="1" visible="yes" active="yes"/>
+<layer number="47" name="Measures" color="7" fill="1" visible="yes" active="yes"/>
+<layer number="48" name="Document" color="7" fill="1" visible="yes" active="yes"/>
+<layer number="49" name="Reference" color="7" fill="1" visible="yes" active="yes"/>
 <layer number="50" name="dxf" color="7" fill="1" visible="no" active="no"/>
-<layer number="51" name="tDocu" color="7" fill="1" visible="no" active="yes"/>
+<layer number="51" name="tDocu" color="7" fill="1" visible="yes" active="yes"/>
 <layer number="52" name="bDocu" color="7" fill="1" visible="yes" active="yes"/>
 <layer number="53" name="tPadExt" color="7" fill="1" visible="no" active="no"/>
@@
 <attribute name="SPICEPREFIX" value="C" x="71.9" y="25.6" size="1.778" layer="27" rot="R270" display="off"/>
 </element>
-<element name="D301" library="BW-Active" library_urn="urn:adsk.eagle:library:33783073" package="SOD323" package3d_urn="urn:adsk.eagle:package:33783196/2" value="NSR0530H" x="73.7" y="31" smashed="yes" rot="R270">
+<element name="D301" library="BW-Active" library_urn="urn:adsk.eagle:library:33783073" package="SOD323" package3d_urn="urn:adsk.eagle:package:33783196/2" value="SS0840WS" x="73.7" y="31" smashed="yes" rot="R270">
 <attribute name="NAME" x="74.8" y="30.4" size="1.016" layer="25" font="vector" ratio="15"/>
 </element>
-<element name="D302" library="BW-Active" library_urn="urn:adsk.eagle:library:33783073" package="SOD323" package3d_urn="urn:adsk.eagle:package:33783196/2" value="NSR0530H" x="73.7" y="27" smashed="yes" rot="R90">
+<element name="D302" library="BW-Active" library_urn="urn:adsk.eagle:library:33783073" package="SOD323" package3d_urn="urn:adsk.eagle:package:33783196/2" value="SS0840WS" x="73.7" y="27" smashed="yes" rot="R90">
 <attribute name="NAME" x="74.8" y="26.5" size="1.016" layer="25" font="vector" ratio="15"/>
-<attribute name="VALUE" x="74.8" y="28.4" size="1.016" layer="27" font="vector" ratio="15"/>
+<attribute name="VALUE" x="74.9" y="28.4" size="1.016" layer="27" font="vector" ratio="15"/>
 </element>
 <element name="C308" library="rcl" library_urn="urn:adsk.eagle:library:334" package="C0603" package3d_urn="urn:adsk.eagle:package:23616/2" value="100nF" x="64.8" y="26.8" smashed="yes" rot="MR90">
@@
 <attribute name="SPICEPREFIX" value="C" x="117.9" y="25.6" size="1.778" layer="27" rot="R270" display="off"/>
 </element>
-<element name="D401" library="BW-Active" library_urn="urn:adsk.eagle:library:33783073" package="SOD323" package3d_urn="urn:adsk.eagle:package:33783196/2" value="NSR0530H" x="119.7" y="31" smashed="yes" rot="R270">
+<element name="D401" library="BW-Active" library_urn="urn:adsk.eagle:library:33783073" package="SOD323" package3d_urn="urn:adsk.eagle:package:33783196/2" value="SS0840WS" x="119.7" y="31" smashed="yes" rot="R270">
 <attribute name="NAME" x="120.8" y="30.4" size="1.016" layer="25" font="vector" ratio="15"/>
 </element>
-<element name="D402" library="BW-Active" library_urn="urn:adsk.eagle:library:33783073" package="SOD323" package3d_urn="urn:adsk.eagle:package:33783196/2" value="NSR0530H" x="119.7" y="27" smashed="yes" rot="R90">
+<element name="D402" library="BW-Active" library_urn="urn:adsk.eagle:library:33783073" package="SOD323" package3d_urn="urn:adsk.eagle:package:33783196/2" value="SS0840WS" x="119.7" y="27" smashed="yes" rot="R90">
 <attribute name="NAME" x="120.8" y="26.5" size="1.016" layer="25" font="vector" ratio="15"/>
-<attribute name="VALUE" x="120.8" y="28.4" size="1.016" layer="27" font="vector" ratio="15"/>
+<attribute name="VALUE" x="120.9" y="28.4" size="1.016" layer="27" font="vector" ratio="15"/>
 </element>
 <element name="C408" library="rcl" library_urn="urn:adsk.eagle:library:334" package="C0603" package3d_urn="urn:adsk.eagle:package:23616/2" value="100nF" x="110.8" y="26.8" smashed="yes" rot="MR90">
@@
 <polygon width="0.1524" layer="1" isolate="1.5">
 <vertex x="5.4" y="30.8"/>
-<vertex x="4.3" y="29.7"/>
-<vertex x="4.3" y="28.3"/>
-<vertex x="5.1" y="27.5"/>
+<vertex x="4.2" y="29.6"/>
+<vertex x="4.2" y="28.2"/>
+<vertex x="4.9" y="27.5"/>
 <vertex x="9.5" y="27.5"/>
 <vertex x="10" y="28"/>
@@
 <vertex x="4.5" y="42.5"/>
 <vertex x="2.5" y="40.5"/>
-<vertex x="2.5" y="27.6"/>
-<vertex x="4.2" y="25.9"/>
+<vertex x="2.5" y="27.4"/>
+<vertex x="4" y="25.9"/>
 <vertex x="24.1" y="25.9"/>
 <vertex x="26" y="24"/>
