File: main.sch (EAGLE design)
At the start: 285 parts, among them J301 12401948E412A, J401 12401948E412A, J501 ICSP, J502 UART, Q101 IPP65R095C7, Q201 IPP65R190C7, Q202 IPP65R190C7, Q203 SiR182DP, Q204 SiR182DP, Q301 ISZ0702NLS, Q302 ISZ0702NLS, Q303 ISZ0702NLS, Q304 ISZ0702NLS, Q401 ISZ0702NLS, Q402 ISZ0702NLS, Q403 ISZ0702NLS, Q404 ISZ0702NLS, T201 706µH 41:4:4:4, U101 UCC28056B, U201 UCC256404, U202 TLV431E5, U203 UCC24624, U301 MAX25432, U401 MAX25432, U501 TPS54308, U502 PIC32MZ-EF-064, U503 LD39150DT33, Y501 24MHz

Commit message: Supply PCB done (?)
Parts:
- added TP101, TP201, TP202, TP301, TP302, TP303, TP304, TP305, TP306, TP401, TP402, TP403, TP404, TP405, TP406, TP501, TP502, TP503, TP504, TP505, TP506, TP507, TP508, TP509: RCU-0(J), BW-PassiveMechanical:RCU-0(J)
- C502, C503, C505, C506, C507, C508, C509, C510, C511, C512: value 0.1µF -> 100nF
Connections:
- net N$1 renamed PIC_UART_TX
- net N$2 renamed PIC_UART_RX
- net 18V: now also TP201.TP
- net 3.3V: now also TP501.TP
- net 3.6V: now also TP509.TP
- net 370V: now also TP101.TP
- net LCD_!CS: now also TP506.TP
- net LCD_!INT: now also TP507.TP
- net LCD_!PD: now also TP508.TP
- net LCD_MISO: now also TP504.TP
- net LCD_MOSI: now also TP505.TP
- net LCD_SCK: now also TP503.TP
- net PIC_VIN_SENSE: now also TP502.TP
- net SGND: now also TP202.TP
- net USB1_!ALERT: now also TP304.TP
- net USB1_CC1: now also TP305.TP
- net USB1_EN: now also TP301.TP
- net USB1_SCL: now also TP302.TP
- net USB1_SDA: now also TP303.TP
- net USB1_VBUS: now also TP306.TP
- net USB2_!ALERT: now also TP404.TP
- net USB2_CC1: now also TP405.TP
- net USB2_EN: now also TP401.TP
- net USB2_SCL: now also TP402.TP
- net USB2_SDA: now also TP403.TP
- net USB2_VBUS: now also TP406.TP
Other:
- moved on the sheet: C401, C402, C403, C404, C405, C406, C407, C408, C409, C410, C411, C412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

Commit message: Base design complete, adapter firmware started
Parts:
- D301, D302, D401, D402: value NSR0530H -> SS0840WS
- U503: device BW-Active:LD39150PU33 -> BW-Active:DFN6-LDO
Changed lines of the file:
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@@
 <part name="C313" library="rcl" library_urn="urn:adsk.eagle:library:334" deviceset="C-EU" device="C0603" package3d_urn="urn:adsk.eagle:package:23616/2" value="100nF"/>
 <part name="C314" library="rcl" library_urn="urn:adsk.eagle:library:334" deviceset="C-EU" device="C0603" package3d_urn="urn:adsk.eagle:package:23616/2" value="100nF"/>
-<part name="D301" library="BW-Active" library_urn="urn:adsk.eagle:library:33783073" deviceset="SOD323-SCHOTTKY" device="" package3d_urn="urn:adsk.eagle:package:33783196/2" value="NSR0530H"/>
-<part name="D302" library="BW-Active" library_urn="urn:adsk.eagle:library:33783073" deviceset="SOD323-SCHOTTKY" device="" package3d_urn="urn:adsk.eagle:package:33783196/2" value="NSR0530H"/>
+<part name="D301" library="BW-Active" library_urn="urn:adsk.eagle:library:33783073" deviceset="SOD323-SCHOTTKY" device="" package3d_urn="urn:adsk.eagle:package:33783196/2" value="SS0840WS"/>
+<part name="D302" library="BW-Active" library_urn="urn:adsk.eagle:library:33783073" deviceset="SOD323-SCHOTTKY" device="" package3d_urn="urn:adsk.eagle:package:33783196/2" value="SS0840WS"/>
 <part name="C308" library="rcl" library_urn="urn:adsk.eagle:library:334" deviceset="C-EU" device="C0603" package3d_urn="urn:adsk.eagle:package:23616/2" value="100nF"/>
 <part name="C305" library="rcl" library_urn="urn:adsk.eagle:library:334" deviceset="C-EU" device="C0603" package3d_urn="urn:adsk.eagle:package:23616/2" value="1µF"/>
@@
 <part name="C514" library="rcl" library_urn="urn:adsk.eagle:library:334" deviceset="C-EU" device="C0805" package3d_urn="urn:adsk.eagle:package:23617/2" value="22µF"/>
 <part name="L501" library="BW-PassiveMechanical" library_urn="urn:adsk.eagle:library:33858467" deviceset="RLB0912" device="" package3d_urn="urn:adsk.eagle:package:33858528/2" value="10µH"/>
-<part name="U503" library="BW-Active" library_urn="urn:adsk.eagle:library:33783073" deviceset="LD39150PU*" device="" package3d_urn="urn:adsk.eagle:package:39954685/2" technology="33" value="LD39150DT33"/>
+<part name="U503" library="BW-Active" library_urn="urn:adsk.eagle:library:33783073" deviceset="DFN6-LDO" device="" package3d_urn="urn:adsk.eagle:package:39954685/2" value="LD39150DT33"/>
 <part name="C517" library="rcl" library_urn="urn:adsk.eagle:library:334" deviceset="C-EU" device="C0805" package3d_urn="urn:adsk.eagle:package:23617/2" value="2.2µF"/>
 <part name="C518" library="rcl" library_urn="urn:adsk.eagle:library:334" deviceset="CPOL-EU" device="D" package3d_urn="urn:adsk.eagle:package:23424/2" value="330µF"/>
@@
 <part name="C413" library="rcl" library_urn="urn:adsk.eagle:library:334" deviceset="C-EU" device="C0603" package3d_urn="urn:adsk.eagle:package:23616/2" value="100nF"/>
 <part name="C414" library="rcl" library_urn="urn:adsk.eagle:library:334" deviceset="C-EU" device="C0603" package3d_urn="urn:adsk.eagle:package:23616/2" value="100nF"/>
-<part name="D401" library="BW-Active" library_urn="urn:adsk.eagle:library:33783073" deviceset="SOD323-SCHOTTKY" device="" package3d_urn="urn:adsk.eagle:package:33783196/2" value="NSR0530H"/>
-<part name="D402" library="BW-Active" library_urn="urn:adsk.eagle:library:33783073" deviceset="SOD323-SCHOTTKY" device="" package3d_urn="urn:adsk.eagle:package:33783196/2" value="NSR0530H"/>
+<part name="D401" library="BW-Active" library_urn="urn:adsk.eagle:library:33783073" deviceset="SOD323-SCHOTTKY" device="" package3d_urn="urn:adsk.eagle:package:33783196/2" value="SS0840WS"/>
+<part name="D402" library="BW-Active" library_urn="urn:adsk.eagle:library:33783073" deviceset="SOD323-SCHOTTKY" device="" package3d_urn="urn:adsk.eagle:package:33783196/2" value="SS0840WS"/>
 <part name="C408" library="rcl" library_urn="urn:adsk.eagle:library:334" deviceset="C-EU" device="C0603" package3d_urn="urn:adsk.eagle:package:23616/2" value="100nF"/>
 <part name="C405" library="rcl" library_urn="urn:adsk.eagle:library:334" deviceset="C-EU" device="C0603" package3d_urn="urn:adsk.eagle:package:23616/2" value="1µF"/>

Commit message: updated
Parts:
- removed C121: 22µF, BW-PassiveMechanical:CPOL-E5-12.5
- removed R114: 59kΩ, rcl:R-US_R0603
- removed R115: 44.2kΩ, rcl:R-US_R0603
- removed RV201: 18V, varistor:VARISTORCN0603
- added D104, D105: S3J, diode:DIODE-SMC
- added D206: 18V, BW-Active:SOD123-ZENER
- added D207: SS16, BW-Active:DO-214AC-SCHOTTKY
- added D208: GS1006FL, BW-Active:SOD123FL-DIODE
- added D209: 15V, BW-Active:SOD123-ZENER
- added D210: 20V, BW-Active:SOD123-ZENER
- added R238, R243: 0Ω, rcl:R-US_R0603
- added R239: 1kΩ, rcl:R-US_R0603
- added R240: 470kΩ, rcl:R-US_R0603
- added R241: 100kΩ, rcl:R-US_R0603
- added R242: 7.5kΩ, rcl:R-US_R0603
- C104: value 470nF -> 10pF 630V; device BW-PassiveMechanical:WCAP-FTX2-470N -> rcl:C-EUC1206
- C105: value 10pF 630V -> 3.9nF; device rcl:C-EUC1206 -> rcl:C-EUC0603
- C106: value 3.9nF -> 470nF; device rcl:C-EUC0603 -> BW-PassiveMechanical:WCAP-FTX2-470N
- C107: value 1µF -> 10µF; device rcl:C-EUC0603 -> rcl:C-EUC0805
- C114: value 0pF 630V -> 22µF; device rcl:C-EUC1206 -> BW-PassiveMechanical:CPOL-E5-12.5
- C204: value 330pF -> 1nF
- C214: value 100nF -> 1µF
- D102: value S3J -> 15V; device diode:DIODE-SMC -> BW-Active:SOD123-ZENER
- D103: value S3J -> 18V; device diode:DIODE-SMC -> BW-Active:SOD123-ZENER
- D203: value SS16 -> GS1006FL; device BW-Active:DO-214AC-SCHOTTKY -> BW-Active:SOD123FL-DIODE
- D205: value 20V -> 18V
- Q201, Q202: value IPP65R190C7 -> IPP65R155CFD7
- R110: value ?Ω -> 3MΩ
- R111, R112: value 4.99MΩ -> 3MΩ
- R113: value 4.99MΩ -> 62kΩ; device rcl:R-US_R1206 -> rcl:R-US_R0603
- R201, R202: value 1Ω -> 47Ω
- R203, R204: value 4.7kΩ -> 1Ω
- R205, R206: value 1.69kΩ -> 4.7kΩ; device rcl:R-US_R1206 -> rcl:R-US_R0603
- R208: value 100Ω -> 4.99MΩ
- R209, R210: value ?Ω -> 4.99MΩ; device rcl:R-US_R0603 -> rcl:R-US_R1206
- R211: value 30kΩ -> 44.2kΩ
- R212: value 0Ω -> 1.69kΩ; device rcl:R-US_R0603 -> rcl:R-US_R1206
- R213: value 5.36kΩ -> 1.69kΩ; device rcl:R-US_R0603 -> rcl:R-US_R1206
- R214: value 0Ω -> 100Ω; device rcl:R-US_R0603 -> rcl:R-US_R1206
- R215: value 1Ω -> ?Ω
- R217: value ?Ω -> 30kΩ
- R218: value 390kΩ -> 0Ω
- R219: value 0Ω -> 5.36kΩ
- R220: value 866kΩ -> 0Ω
- R221: value 0Ω -> 1Ω
- R224: value 1kΩ -> 390kΩ
- R226: value 1kΩ -> 866kΩ
- R228, R229: value 0Ω -> ?Ω
- R230: value ?Ω -> 1kΩ
- R231: value 100Ω -> 0Ω
- R232: value 0Ω -> 1kΩ
- R233: value 1kΩ -> 0Ω
- R234: value 470kΩ -> 0Ω
- R235: value 100kΩ -> 0Ω
- R236: value 7.5kΩ -> ?Ω
- R237: value 0Ω -> 100Ω
Connections:
- removed net PFC_SNUBBER: C114.1, R110.1
- new net LLC_BLK_RB: R209.1, R210.2
- new net LLC_BLK_RT: R208.1, R209.2
- new net LLC_HO_DIS: D201.A, R203.1
- new net LLC_LO_DIS: D202.A, R204.1
- net 18V: now also D210.C; no longer RV201.1
- net 370V: now also C114.+, R110.2, R208.2; no longer C121.+, R111.2
- net AC_L_FILTERED: now also C106.1, D203.A; no longer C104.1, D201.A
- net AC_N_FILTERED: now also C106.2, D204.A; no longer C104.2, D202.A
- net AC_RECTIFIED: now also D104.A; no longer D102.A
- net LLC_AUX: now also D207.A, R215.2, R217.2; no longer D203.A, R209.2, R211.2
- net LLC_BLK: now also R210.1, R211.2; no longer R114.1, R115.2
- net LLC_BW: now also R216.2, R218.1, R219.2; no longer R210.2, R212.1, R213.2
- net LLC_BW_RB: now also R216.1, R219.1, R220.2; no longer R210.1, R213.1, R214.2
- net LLC_BW_RT: now also R215.1, R217.1, R218.2; no longer R209.1, R211.1, R212.2
- net LLC_FB_COMP: now also R236.2, R237.2; no longer R230.2, R231.2
- net LLC_FB_COMPR: now also R235.2, R236.1, R237.1; no longer R229.2, R230.1, R231.1
- net LLC_FB_OPA: now also R229.2, R231.1, R232.2; no longer R223.2, R225.1, R226.2
- net LLC_FB_OPAP: now also D209.C, R228.2, R230.2, R239.1; no longer D205.C, R222.2, R224.2, R233.1
- net LLC_FB_OPAR: now also R228.1, R230.1, R231.2; no longer R222.1, R224.1, R225.2
- net LLC_FB_OPBR: now also R229.1, R232.1, R233.2; no longer R223.1, R226.1, R227.2
- net LLC_FB_OPK: now also R233.1, R235.1; no longer R227.1, R229.1
- net LLC_FB_VREF: now also R240.2, R241.1, R242.2; no longer R234.2, R235.1, R236.2
- net LLC_FB_VREFR: now also R240.1, R242.1, R243.2; no longer R234.1, R236.1, R237.2
- net LLC_HB: now also D208.C; no longer D204.C
- net LLC_HB_FEED: now also D208.A, R221.1; no longer D204.A, R215.1
- net LLC_HO: now also D201.C
- net LLC_HO_R: now also D205.C, R205.2
- net LLC_HS: now also D205.A, R205.1; no longer R203.1
- net LLC_HV: now also R213.2; no longer R207.2
- net LLC_HV_RB: now also R212.2, R213.1; no longer R206.2, R207.1
- net LLC_HV_RECT: now also D203.C, D204.C, R207.1; no longer D201.C, D202.C, R205.1
- net LLC_HV_RT: now also R207.2, R212.1; no longer R205.2, R206.1
- net LLC_ISNS: now also R214.2; no longer R208.2
- net LLC_LL/SS: now also R223.2, R225.1, R226.2; no longer R217.2, R219.1, R220.2
- net LLC_LL_RB: now also R223.1, R226.1, R227.2; no longer R217.1, R220.1, R221.2
- net LLC_LL_RT: now also R222.1, R224.1, R225.2; no longer R216.1, R218.1, R219.2
- net LLC_LO: now also D202.C
- net LLC_LO_R: now also D206.C, R206.2
- net LLC_OUT: now also R239.2, R241.2; no longer R233.2, R235.2
- net LLC_RVCC: now also R221.2, R222.2, R224.2; no longer R215.2, R216.2, R218.2
- net LLC_SR_VG1: now also R234.2; no longer R228.2
- net LLC_SR_VG1_R: now also R234.1; no longer R228.1
- net LLC_SR_VG2: now also R238.1; no longer R232.1
- net LLC_SR_VG2_R: now also R238.2; no longer R232.2
- net LLC_VCC: now also D207.C; no longer D203.C
- net PFC_CS: now also C105.2, D103.A; no longer C106.2
- net PFC_DRV_R: now also D103.C
- net PFC_OUT_RAW: now also D104.C, D105.C; no longer D102.C, D103.C
- net PFC_SW_NODE: now also C104.1, D105.A; no longer C105.1, D103.A, R110.2
- net PFC_VCC: now also D102.C
- net PFC_VOSNS: now also R112.1, R113.2; no longer R113.1, R114.2
- net PFC_VOSNS_RB: now also R111.1, R112.2; no longer R112.1, R113.2
- net PFC_VOSNS_RT: now also R110.1, R111.2; no longer R111.1, R112.2
- net PFC_ZCD/CS_RAW: now also C104.2, C105.1; no longer C105.2, C106.1
- net PGND: now also C114.-, D102.A, D206.A, R113.1, R206.1, R211.1, R220.1, R227.1; no longer C114.2, C121.-, R115.1, R204.1, R208.1, R221.1
- net SGND: now also D209.A, D210.A, R243.1; no longer D205.A, R237.1, RV201.2
Other:
- moved on the sheet: C104, C105, C106, C115, C116, C117, C118, C119, C120, D101, D102, D103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
